File: hardware/sensor_auxiliary/sensor_auxiliary.sch (KiCad schematic (older format))
At the start: 12 parts, among them J1 Conn_01x02, J2 Conn_01x02, J3 Conn_01x02, U1 QRE1113

Commit message: Relayout for 2 SPI master lines, finished 14 and 15 sensor boards, finished auxiliary board
Parts:
- removed C5, C6: 100nF, Capacitor_SMD:C_0805_2012Metric_Pad1.15x1.40mm_HandSolder, symbol Device:C_Small
- removed C7, C8: 10uF, Capacitor_Tantalum_SMD:CP_EIA-2012-15_AVX-P_Pad1.30x1.05mm_HandSolder, symbol Device:CP_Small
- removed J1, J2, J3: Conn_01x02, Connector_PinHeader_2.54mm:PinHeader_1x02_P2.54mm_Horizontal, symbol Connector_Generic:Conn_01x02
- added C2: 10uF, Capacitor_Tantalum_SMD:CP_EIA-2012-15_AVX-P_Pad1.30x1.05mm_HandSolder, symbol Device:CP_Small
- added C3: 100nF, Capacitor_SMD:C_0805_2012Metric_Pad1.15x1.40mm_HandSolder, symbol Device:C_Small
- added H1, H2, H3, H4: M2, MountingHole:MountingHole_2.2mm_M2_Pad_Via, symbol Mechanical:MountingHole_Pad
- added J1: Conn_01x04, Connector_FFC-FPC:Molex_200528-0040_1x04-1MP_P1.00mm_Horizontal, symbol Connector_Generic:Conn_01x04
- renumbered R3 to R2
Connections:
- wire segments 51 -> 49
Other:
- note added: "Connector"
- note added: "Mounting Holes"
- note added: "Power Buffer"
- note removed: "Power Header L"
- note removed: "Power Header R"
- note removed: "Sensor Header"
