File: hardware/sensor_auxiliary/sensor_auxiliary.kicad_pcb (KiCad board)
At the start: 2 copper layers, 25 x 25 mm, 12 parts, among them J1 Conn_01x04, U1 QRE1113

Commit message: Created main controller. Prototypes finished.
Parts:
- added REF**: OpKey_Logo, OpKey:OpKey_Logo, B.Cu at (43.1, 37.8)
- added REF**: OSHW-Logo2_9.8x8mm_SilkScreen, Symbol:OSHW-Logo2_9.8x8mm_SilkScreen, B.Cu at (42.3, 48.8)
Routing:
- net GND: track 43.3 -> 48.4 mm
Other:
- board text added: "Auxiliary Optical Sensor"
- board text added: "OPKEY"
