File: hardware/sensor_auxiliary/sensor_auxiliary.kicad_pcb (KiCad board)
At the start: 2 copper layers, 25 x 25 mm, 14 parts, among them J1 Conn_01x04, U1 QRE1113

Commit message: Final changes, regenerated gerber files
Other:
- board text added: "JLCJLCJLCJLC"
Changed lines of the file:
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@@
   (general
     (thickness 1.6)
-    (drawings 6)
+    (drawings 7)
     (tracks 26)
     (zones 0)
@@
       (viasonmask false)
       (mode 1)
-      (useauxorigin false)
+      (useauxorigin true)
       (hpglpennumber 1)
       (hpglpenspeed 20)
@@
     )
   )
+  (gr_text JLCJLCJLCJLC (at 31.5 42.5 270) (layer B.SilkS)
+    (effects (font (size 1.5 1.5) (thickness 0.3)) (justify mirror))
+  )
   (gr_text "Auxiliary Optical Sensor" (at 31.6 42.5 90) (layer F.SilkS)
