File: hardware/main_controller/main_controller.kicad_pcb (KiCad board)
At the start: 2 copper layers, 70 x 40 mm, 39 parts, among them J1 Conn_01x17, J2 Conn_01x17, J3 Barrel_Jack, J4 Conn_01x02, J5 Conn_01x04, J6 Conn_01x04, J7 USB_B_Micro, J8 Conn_01x03, J9 Conn_01x03, Q1 2N7002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

Commit message: Final changes, regenerated gerber files
Other:
- board text added: "JLCJLCJLCJLC"
- board text added: "Type A"
- board text added: "Type B"
- board text removed: "Type L"
- board text removed: "Type R"
