File: hardware/sensor_array_13_sensors/sensor_array_13_sensors.kicad_pcb (KiCad board)
At the start: 2 copper layers, 180 x 30 mm, 86 parts, among them J1 Conn_01x17, J2 Conn_01x17, J3 Conn_01x04, J4 Conn_01x04, J5 Conn_01x03, J6 Conn_01x04, J7 Conn_01x04, U10 QRE1113, U11 QRE1113, U12 QRE1113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

Commit message: Created main controller. Prototypes finished.
Parts:
- added REF**: OpKey_Logo, OpKey:OpKey_Logo, F.Cu at (52.0, 36.0)
- moved REF** 70.9 mm to (121.5, 49.4)
Changed lines of the file:
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@@
     (tracks 757)
     (zones 0)
-    (modules 86)
+    (modules 87)
     (nets 60)
   )
@@
     (add_net SDO1)
   )
+  (module OpKey:OpKey_Logo locked (layer F.Cu)
+    (at 52 36)
+    (attr virtual)
+    (fp_text reference REF** (at 0 8.4) (layer F.SilkS) hide
+      (effects (font (size 1 1) (thickness 0.15)))
+    )
+    (fp_text value OpKey_Logo (at 0 7.4) (layer F.Fab) hide
+      (effects (font (size 1 1) (thickness 0.15)))
+    )
+    (fp_text user OPKEY (at 0 1.8) (layer F.SilkS)
+      (effects (font (size 1.5 1.5) (thickness 0.3)))
+    )
+    (fp_line (start -1 -2.8) (end -2 -3.8) (layer F.SilkS) (width 0.2))
+    (fp_line (start -2 -3.8) (end -1.8 -3.1) (layer F.SilkS) (width 0.2))
+    (fp_line (start -2 -3.8) (end -1.3 -3.6) (layer F.SilkS) (width 0.2))
+    (fp_line (start -3.3 -3.3) (end -2.6 -3.1) (layer F.SilkS) (width 0.2))
+    (fp_line (start -3.3 -3.3) (end -3.1 -2.6) (layer F.SilkS) (width 0.2))
+    (fp_line (start -2.3 -2.3) (end -3.3 -3.3) (layer F.SilkS) (width 0.2))
+    (fp_line (start -1.8 -1.15) (end -3 -1.15) (layer F.SilkS) (width 0.2))
+    (fp_line (start -1.8 -0.15) (end -1.8 -1.15) (layer F.SilkS) (width 0.12))
+    (fp_line (start -1.8 -2.15) (end -1.8 -0.15) (layer F.SilkS) (width 0.2))
+    (fp_line (start -1.8 -1.15) (end 0.2 -0.15) (layer F.SilkS) (width 0.2))
+    (fp_line (start 0.2 -2.15) (end -1.8 -1.15) (layer F.SilkS) (width 0.2))
+    (fp_line (start 0.2 -0.15) (end 0.2 -2.15) (layer F.SilkS) (width 0.2))
+    (fp_line (start 1.4 -1.15) (end 0.2 -1.15) (layer F.SilkS) (width 0.2))
+    (fp_line (start 4.5 3) (end 4 3.5) (layer F.SilkS) (width 0.12))
+    (fp_line (start 3.75 3) (end 3.25 3.5) (layer F.SilkS) (width 0.12))
+    (fp_line (start 3 3) (end 2.5 3.5) (layer F.SilkS) (width 0.12))
+    (fp_line (start 0.75 3) (end 0.25 3.5) (layer F.SilkS) (width 0.12))
+    (fp_line (start 0 3) (end -0.5 3.5) (layer F.SilkS) (width 0.12))
+    (fp_line (start 1.5 3) (end 1 3.5) (layer F.SilkS) (width 0.12))
+    (fp_line (start -0.75 3) (end -1.25 3.5) (layer F.SilkS) (width 0.12))
+    (fp_line (start 2.25 3) (end 1.75 3.5) (layer F.SilkS) (width 0.12))
+    (fp_arc (start 3.75 -1) (end 2.5 -1) (angle -90) (layer F.SilkS) (width 0.12))
+    (fp_arc (start 3.75 1.5) (end 5 1.5) (angle -90) (layer F.SilkS) (width 0.12))
+    (fp_arc (start -1.25 -1) (end 2.5 -1) (angle -180) (layer F.SilkS) (width 0.12))
+    (fp_line (start 5 3.5) (end 5 1.5) (layer F.SilkS) (width 0.12))
+    (fp_line (start 4.5 3.5) (end 5 3.5) (layer F.SilkS) (width 0.12))
+    (fp_line (start -5 3.5) (end -5 -1) (layer F.SilkS) (width 0.12))
+    (fp_line (start -4.5 3.5) (end -5 3.5) (layer F.SilkS) (width 0.12))
+    (fp_poly (pts (xy 3.25 4.5) (xy 3.25 3.5) (xy 3.75 3.5) (xy 3.75 4.5)) (layer F.SilkS) (width 0.1))
+    (fp_poly (pts (xy 2.25 4.5) (xy 2.25 3.5) (xy 2.75 3.5) (xy 2.75 4.5)) (layer F.SilkS) (width 0.1))
+    (fp_poly (pts (xy 0.75 4.5) (xy 0.75 3.5) (xy 1.25 3.5) (xy 1.25 4.5)) (layer F.SilkS) (width 0.1))
+    (fp_poly (pts (xy -0.25 4.5) (xy -0.25 3.5) (xy 0.25 3.5) (xy 0.25 4.5)) (layer F.SilkS) (width 0.1))
+    (fp_poly (pts (xy -1.25 4.5) (xy -1.25 3.5) (xy -0.75 3.5) (xy -0.75 4.5)) (layer F.SilkS) (width 0.1))
+    (fp_poly (pts (xy -2.75 4.5) (xy -2.75 3.5) (xy -2.25 3.5) (xy -2.25 4.5)) (layer F.SilkS) (width 0.1))
+    (fp_poly (pts (xy -3.75 4.5) (xy -3.75 3.5) (xy -3.25 3.5) (xy -3.25 4.5)) (layer F.SilkS) (width 0.1))
+    (fp_line (start 4.5 5) (end 4.5 3.5) (layer F.SilkS) (width 0.12))
+    (fp_line (start -4.5 5) (end 4.5 5) (layer F.SilkS) (width 0.12))
+    (fp_line (start -4.5 3.5) (end -4.5 5) (layer F.SilkS) (width 0.12))
+    (fp_line (start 4.5 3.5) (end -4.5 3.5) (layer F.SilkS) (width 0.12))
+    (fp_line (start -4.5 3) (end -5 3.5) (layer F.SilkS) (width 0.12))
+    (fp_line (start -3.75 3) (end -4.25 3.5) (layer F.SilkS) (width 0.12))
+    (fp_line (start -3 3) (end -3.5 3.5) (layer F.SilkS) (width 0.12))
+    (fp_line (start -2.25 3) (end -2.75 3.5) (layer F.SilkS) (width 0.12))
+    (fp_line (start -1.5 3) (end -2 3.5) (layer F.SilkS) (width 0.12))
+  )
   (module Symbol:OSHW-Logo2_9.8x8mm_SilkScreen locked (layer F.Cu)
-    (at 52 35.3)
+    (at 121.5 49.4)
     (descr "Open Source Hardware Symbol")
     (tags "Logo Symbol OSHW")
@@
     (tags "Potentiometer Bourns TC33X Vertical")
     (attr smd)
-    (fp_text reference RV3 (at 0 -2.5) (layer F.SilkS)
+    (fp_text reference RV3 (at -0.003333 2.6) (layer F.SilkS)
       (effects (font (size 1 1) (thickness 0.15)))
     )
@@
     (tags SOT-23)
     (attr smd)
-    (fp_text reference U17 (at 2.3 0 90) (layer F.SilkS)
+    (fp_text reference U17 (at 1 -2.5 180) (layer F.SilkS)
       (effects (font (size 1 1) (thickness 0.15)))
     )
@@
     (tags "capacitor handsolder")
     (attr smd)
-    (fp_text reference C18 (at 2.3 0 270) (layer F.SilkS)
+    (fp_text reference C18 (at 0 1.5) (layer F.SilkS)
       (effects (font (size 1 1) (thickness 0.15)))
     )
@@
   (gr_line (start 151.6 45.2) (end 151.6 35.2) (layer F.SilkS) (width 0.12))
   (gr_line (start 148.4 45.2) (end 148.4 35.2) (layer F.SilkS) (width 0.12))
-  (gr_text 1 (at 144.2 39.2 90) (layer F.SilkS)
+  (gr_text 0 (at 144.2 39.2 90) (layer F.SilkS)
     (effects (font (size 1 1) (thickness 0.15)))
   )
-  (gr_text 0 (at 144.2 43.2 90) (layer F.SilkS)
+  (gr_text 1 (at 144.2 43.2 90) (layer F.SilkS)
     (effects (font (size 1 1) (thickness 0.15)))
   )
