File: hardware/sensor_array_13_sensors/sensor_array_13_sensors.kicad_pcb (KiCad board)
At the start: 2 copper layers, 180 x 30 mm, 87 parts, among them J1 Conn_01x17, J2 Conn_01x17, J3 Conn_01x04, J4 Conn_01x04, J5 Conn_01x03, J6 Conn_01x04, J7 Conn_01x04, U10 QRE1113, U11 QRE1113, U12 QRE1113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

Commit message: Final changes, regenerated gerber files
Parts:
- JP1, JP10, JP11, JP12, JP2, JP3, JP4, JP5, JP6, JP7, JP8, JP9: footprint Jumper:SolderJumper-2_P1.3mm_Open_RoundedPad1.0x1.5mm -> OpKey:SolderJumper-2_P1.3mm_Open_RoundedPad1.0x1.5mm
Other:
- board text added: "JLCJLCJLCJLC"
- board text added: "Type A"
- board text added: "Type B"
