File: hardware/sensor_array_15_sensors/sensor_array_15_sensors.kicad_pcb (KiCad board)
At the start: 2 copper layers, 205 x 30 mm, 83 parts, among them J1 Conn_01x17, J2 Conn_01x17, J3 Conn_01x04, J4 Conn_01x04, J5 Conn_01x02, U1 QRE1113, U10 QRE1113, U11 QRE1113, U12 QRE1113, U13 QRE1113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

Commit message: Relayout for 2 SPI master lines, finished 14 and 15 sensor boards, finished auxiliary board
Parts:
- added JP10: SDO, Jumper:SolderJumper-2_P1.3mm_Open_RoundedPad1.0x1.5mm, F.Cu at (189.6, 43.2)
- added JP11: SDO, Jumper:SolderJumper-2_P1.3mm_Open_RoundedPad1.0x1.5mm, F.Cu at (192.8, 39.2)
- added JP12: SDO, Jumper:SolderJumper-2_P1.3mm_Open_RoundedPad1.0x1.5mm, F.Cu at (192.8, 43.2)
- added JP7: SDO, Jumper:SolderJumper-2_P1.3mm_Open_RoundedPad1.0x1.5mm, F.Cu at (186.4, 39.2)
- added JP8: SDO, Jumper:SolderJumper-2_P1.3mm_Open_RoundedPad1.0x1.5mm, F.Cu at (186.4, 43.2)
- added JP9: SDO, Jumper:SolderJumper-2_P1.3mm_Open_RoundedPad1.0x1.5mm, F.Cu at (189.6, 39.2)
- added REF**: OSHW-Logo2_9.8x8mm_SilkScreen, Symbol:OSHW-Logo2_9.8x8mm_SilkScreen, F.Cu at (52.0, 35.3)
- J5: value Conn_01x02 -> Conn_01x03; footprint Connector_PinHeader_2.54mm:PinHeader_1x02_P2.54mm_Horizontal -> Connector_PinHeader_2.54mm:PinHeader_1x03_P2.54mm_Horizontal
- moved JP3 32.1 mm to (178.2, 39.2)
- moved JP2 31.6 mm to (175.0, 39.2)
- moved JP1 31.0 mm to (171.8, 39.2)
- moved JP6 23.6 mm to (178.2, 43.2)
- moved JP5 23.0 mm to (175.0, 43.2)
- moved JP4 22.5 mm to (171.8, 43.2)
- moved C22 9.19 mm to (117.9, 39.6)
- moved C20 4.88 mm to (127.0, 39.6), turned to 0 degrees
- moved C23 4.60 mm to (122.2, 39.6), turned to 180 degrees
- moved J4 3.61 mm to (156.8, 41.2), turned to 180 degrees
- moved J5 3.50 mm to (209.3, 41.3)
- moved R1 2.50 mm to (58.1, 47.7)
- moved RV1 2.50 mm to (52.6, 47.7)
- moved C18 1.20 mm to (139.2, 48.6), turned to 0 degrees
Connections:
- J1 pad 1: SCLK -> +5V
- J1 pad 10: GND -> CS5
- J1 pad 11: GND -> CS4
- J1 pad 12: +3V3 -> CS3
- J1 pad 13: GND -> CS2
- J1 pad 14: +5V -> CS1
- J1 pad 15: GND -> CS0
- J1 pad 16: +5V -> +3V3
- J1 pad 17: GND -> +5V
- J1 pad 2: SDI -> SCLK1
- J1 pad 3: SDO -> SDI1
- J1 pad 4: CS5 -> SDO1
- J1 pad 5: CS4 -> GND
- J1 pad 6: CS3 -> SCLK0
- J1 pad 7: CS2 -> SDI0
- J1 pad 8: CS1 -> SDO0
- J1 pad 9: CS0 -> GND
- J2 pad 1: GND -> +5V
- J2 pad 10: CS1 -> SDO0
- J2 pad 11: CS2 -> SDI0
- J2 pad 12: CS3 -> SCLK0
- J2 pad 13: CS4 -> GND
- J2 pad 14: CS5 -> SDO1
- J2 pad 15: SDO -> SDI1
- J2 pad 16: SDI -> SCLK1
- J2 pad 17: SCLK -> +5V
- J2 pad 2: +5V -> +3V3
- J2 pad 3: GND -> CS0
- J2 pad 4: +5V -> CS1
- J2 pad 5: GND -> CS2
- J2 pad 6: +3V3 -> CS3
- J2 pad 7: GND -> CS4
- J2 pad 8: GND -> CS5
- J2 pad 9: CS0 -> GND
Routing:
- net GND: track 191.3 -> 406.8 mm
- net SDO1: track 0.00 -> 204.0 mm, vias 0 -> 2
- net SDI1: track 0.00 -> 201.6 mm, vias 0 -> 2
- net SCLK1: track 0.00 -> 199.0 mm, vias 0 -> 2
- net SDO0: track 0.00 -> 194.4 mm, vias 0 -> 2
- net SDI0: track 0.00 -> 192.0 mm, vias 0 -> 2
- net SCLK0: track 0.00 -> 191.9 mm, vias 0 -> 2
- net SDO: track 195.8 -> 58.3 mm, vias 2 -> 0
- net SDI: track 196.5 -> 61.7 mm, vias 2 -> 0
- net SCLK: track 197.5 -> 65.1 mm, vias 2 -> 0
- net CS: track 20.1 -> 58.1 mm, vias 0 -> 2
- net +5V: track 101.0 -> 112.0 mm
- net +3V3: track 204.4 -> 193.7 mm, vias 0 -> 2
- net CS3: track 195.6 -> 203.2 mm
- net CS4: track 194.5 -> 200.7 mm
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- added copper zone on F.Cu, net +3V3
Other:
- board text added: "CS SEL"
- board text added: "CS line"
- board text added: "OPKEY"
- board text added: "Optical Sensor Array"
- board text added: "SPI SEL"
- board text added: "SPI line"
- board text removed: "3"
- board text removed: "4"
- board text removed: "5"
- board text removed: "CS selector"

Commit message: Created main controller. Prototypes finished.
Parts:
- added REF**: OpKey_Logo, OpKey:OpKey_Logo, F.Cu at (52.0, 36.0)
- moved REF** 95.5 mm to (146.5, 49.4)
Changed lines of the file:
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@@
     (tracks 768)
     (zones 0)
-    (modules 90)
+    (modules 91)
     (nets 62)
   )
@@
   )
   (setup
-    (last_trace_width 0.3)
+    (last_trace_width 0.5)
     (user_trace_width 0.2)
     (user_trace_width 0.3)
@@
     (add_net SDO1)
   )
+  (module OpKey:OpKey_Logo locked (layer F.Cu)
+    (at 52 36)
+    (attr virtual)
+    (fp_text reference REF** (at 0 8.4) (layer F.SilkS) hide
+      (effects (font (size 1 1) (thickness 0.15)))
+    )
+    (fp_text value OpKey_Logo (at 0 7.4) (layer F.Fab) hide
+      (effects (font (size 1 1) (thickness 0.15)))
+    )
+    (fp_text user OPKEY (at 0 1.8) (layer F.SilkS)
+      (effects (font (size 1.5 1.5) (thickness 0.3)))
+    )
+    (fp_line (start -1 -2.8) (end -2 -3.8) (layer F.SilkS) (width 0.2))
+    (fp_line (start -2 -3.8) (end -1.8 -3.1) (layer F.SilkS) (width 0.2))
+    (fp_line (start -2 -3.8) (end -1.3 -3.6) (layer F.SilkS) (width 0.2))
+    (fp_line (start -3.3 -3.3) (end -2.6 -3.1) (layer F.SilkS) (width 0.2))
+    (fp_line (start -3.3 -3.3) (end -3.1 -2.6) (layer F.SilkS) (width 0.2))
+    (fp_line (start -2.3 -2.3) (end -3.3 -3.3) (layer F.SilkS) (width 0.2))
+    (fp_line (start -1.8 -1.15) (end -3 -1.15) (layer F.SilkS) (width 0.2))
+    (fp_line (start -1.8 -0.15) (end -1.8 -1.15) (layer F.SilkS) (width 0.12))
+    (fp_line (start -1.8 -2.15) (end -1.8 -0.15) (layer F.SilkS) (width 0.2))
+    (fp_line (start -1.8 -1.15) (end 0.2 -0.15) (layer F.SilkS) (width 0.2))
+    (fp_line (start 0.2 -2.15) (end -1.8 -1.15) (layer F.SilkS) (width 0.2))
+    (fp_line (start 0.2 -0.15) (end 0.2 -2.15) (layer F.SilkS) (width 0.2))
+    (fp_line (start 1.4 -1.15) (end 0.2 -1.15) (layer F.SilkS) (width 0.2))
+    (fp_line (start 4.5 3) (end 4 3.5) (layer F.SilkS) (width 0.12))
+    (fp_line (start 3.75 3) (end 3.25 3.5) (layer F.SilkS) (width 0.12))
+    (fp_line (start 3 3) (end 2.5 3.5) (layer F.SilkS) (width 0.12))
+    (fp_line (start 0.75 3) (end 0.25 3.5) (layer F.SilkS) (width 0.12))
+    (fp_line (start 0 3) (end -0.5 3.5) (layer F.SilkS) (width 0.12))
+    (fp_line (start 1.5 3) (end 1 3.5) (layer F.SilkS) (width 0.12))
+    (fp_line (start -0.75 3) (end -1.25 3.5) (layer F.SilkS) (width 0.12))
+    (fp_line (start 2.25 3) (end 1.75 3.5) (layer F.SilkS) (width 0.12))
+    (fp_arc (start 3.75 -1) (end 2.5 -1) (angle -90) (layer F.SilkS) (width 0.12))
+    (fp_arc (start 3.75 1.5) (end 5 1.5) (angle -90) (layer F.SilkS) (width 0.12))
+    (fp_arc (start -1.25 -1) (end 2.5 -1) (angle -180) (layer F.SilkS) (width 0.12))
+    (fp_line (start 5 3.5) (end 5 1.5) (layer F.SilkS) (width 0.12))
+    (fp_line (start 4.5 3.5) (end 5 3.5) (layer F.SilkS) (width 0.12))
+    (fp_line (start -5 3.5) (end -5 -1) (layer F.SilkS) (width 0.12))
+    (fp_line (start -4.5 3.5) (end -5 3.5) (layer F.SilkS) (width 0.12))
+    (fp_poly (pts (xy 3.25 4.5) (xy 3.25 3.5) (xy 3.75 3.5) (xy 3.75 4.5)) (layer F.SilkS) (width 0.1))
+    (fp_poly (pts (xy 2.25 4.5) (xy 2.25 3.5) (xy 2.75 3.5) (xy 2.75 4.5)) (layer F.SilkS) (width 0.1))
+    (fp_poly (pts (xy 0.75 4.5) (xy 0.75 3.5) (xy 1.25 3.5) (xy 1.25 4.5)) (layer F.SilkS) (width 0.1))
+    (fp_poly (pts (xy -0.25 4.5) (xy -0.25 3.5) (xy 0.25 3.5) (xy 0.25 4.5)) (layer F.SilkS) (width 0.1))
+    (fp_poly (pts (xy -1.25 4.5) (xy -1.25 3.5) (xy -0.75 3.5) (xy -0.75 4.5)) (layer F.SilkS) (width 0.1))
+    (fp_poly (pts (xy -2.75 4.5) (xy -2.75 3.5) (xy -2.25 3.5) (xy -2.25 4.5)) (layer F.SilkS) (width 0.1))
+    (fp_poly (pts (xy -3.75 4.5) (xy -3.75 3.5) (xy -3.25 3.5) (xy -3.25 4.5)) (layer F.SilkS) (width 0.1))
+    (fp_line (start 4.5 5) (end 4.5 3.5) (layer F.SilkS) (width 0.12))
+    (fp_line (start -4.5 5) (end 4.5 5) (layer F.SilkS) (width 0.12))
+    (fp_line (start -4.5 3.5) (end -4.5 5) (layer F.SilkS) (width 0.12))
+    (fp_line (start 4.5 3.5) (end -4.5 3.5) (layer F.SilkS) (width 0.12))
+    (fp_line (start -4.5 3) (end -5 3.5) (layer F.SilkS) (width 0.12))
+    (fp_line (start -3.75 3) (end -4.25 3.5) (layer F.SilkS) (width 0.12))
+    (fp_line (start -3 3) (end -3.5 3.5) (layer F.SilkS) (width 0.12))
+    (fp_line (start -2.25 3) (end -2.75 3.5) (layer F.SilkS) (width 0.12))
+    (fp_line (start -1.5 3) (end -2 3.5) (layer F.SilkS) (width 0.12))
+  )
   (module Connector_FFC-FPC:Molex_200528-0170_1x17-1MP_P1.00mm_Horizontal locked (layer F.Cu)
     (at 44 42.8 270)
@@
   )
   (module Symbol:OSHW-Logo2_9.8x8mm_SilkScreen locked (layer F.Cu)
-    (at 52 35.3)
+    (at 146.5 49.4)
     (descr "Open Source Hardware Symbol")
     (tags "Logo Symbol OSHW")
@@
     (tags "Potentiometer Bourns TC33X Vertical")
     (attr smd)
-    (fp_text reference RV3 (at 0 -2.5) (layer F.SilkS)
+    (fp_text reference RV3 (at 0 2.6) (layer F.SilkS)
       (effects (font (size 1 1) (thickness 0.15)))
     )
@@
     (tags SOT-23)
     (attr smd)
-    (fp_text reference U17 (at 2.3 0 90) (layer F.SilkS)
+    (fp_text reference U17 (at 1 -2.5 180) (layer F.SilkS)
       (effects (font (size 1 1) (thickness 0.15)))
     )
@@
     (tags "capacitor handsolder")
     (attr smd)
-    (fp_text reference C18 (at 2.3 0 270) (layer F.SilkS)
+    (fp_text reference C18 (at 0 1.5) (layer F.SilkS)
       (effects (font (size 1 1) (thickness 0.15)))
     )
@@
   (gr_line (start 176.6 45.2) (end 176.6 35.2) (layer F.SilkS) (width 0.12))
   (gr_line (start 173.4 45.2) (end 173.4 35.2) (layer F.SilkS) (width 0.12))
-  (gr_text 1 (at 169.2 39.2 90) (layer F.SilkS)
+  (gr_text 0 (at 169.2 39.2 90) (layer F.SilkS)
     (effects (font (size 1 1) (thickness 0.15)))
   )
-  (gr_text 0 (at 169.2 43.2 90) (layer F.SilkS)
+  (gr_text 1 (at 169.2 43.2 90) (layer F.SilkS)
     (effects (font (size 1 1) (thickness 0.15)))
   )
