File: hardware/sensor_array_15_sensors/sensor_array_15_sensors.sch (KiCad schematic (older format))
At the start: 83 parts, among them J1 Conn_01x17, J2 Conn_01x17, J3 Conn_01x04, J4 Conn_01x04, J5 Conn_01x02, U1 QRE1113, U10 QRE1113, U11 QRE1113, U12 QRE1113, U13 QRE1113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

Commit message: Relayout for 2 SPI master lines, finished 14 and 15 sensor boards, finished auxiliary board
Parts:
- added JP10, JP11, JP12, JP7, JP8, JP9: SDO, Jumper:SolderJumper-2_P1.3mm_Open_RoundedPad1.0x1.5mm, symbol Jumper:SolderJumper_2_Open
- J5: value Conn_01x02 -> Conn_01x03; footprint Connector_PinHeader_2.54mm:PinHeader_1x02_P2.54mm_Horizontal -> Connector_PinHeader_2.54mm:PinHeader_1x03_P2.54mm_Horizontal; symbol Connector_Generic:Conn_01x02 -> Connector_Generic:Conn_01x03
Connections:
- net labels added: SCLK0, SCLK1, SDI0, SDI1, SDO0, SDO1
- wire segments 428 -> 436
Other:
- note added: "SPI Line Select"
- moved on the sheet: C20, C21, JP6

Commit message: Created main controller. Prototypes finished.
Parts:
- U16: symbol opmc:ADS7953 -> OpKey:ADS7953
Changed lines of the file:
@@
 EESchema Schematic File Version 4
 LIBS:sensor_array_15_sensors-cache
-LIBS:sensor_array_13_sensors-cache
 EELAYER 29 0
 EELAYER END
@@
 $EndComp
 $Comp
-L opmc:ADS7953 U16
+L OpKey:ADS7953 U16
 U 1 1 5D407382
 P 7300 2500
